Commit message: added camera launch

File: description/robot_base.urdf.xacro (robot description, xacro)
@@ -10,5 +10,13 @@
 	      <color rgba="0.0 0.8 0.0 1.0"/>
 	    </material>
-	  <!-- REMOVED base_footprint is a fictitious link(frame) that is on the ground right below base_link origin, navigation stack depends on this frame -->
+	  <!-- base_footprint is a fictitious link(frame) that is on the ground right below base_link origin, navigation stack depends on this frame -->
+    <!-- BASE_FOOTPRINT LINK -->
+    <joint name="base_footprint_joint" type="fixed">
+        <parent link="base_link"/>
+        <child link="base_footprint"/>
+        <origin xyz="0 0 0" rpy="0 0 0"/>
+    </joint>
+    <link name="base_footprint">
+    </link>
 	  <link name="base_link">
 	    <inertial>
@@ -137,5 +145,7 @@
 	    <axis xyz="0 1 0"/>
 	  </joint>
-	  <joint name="gyro_joint" type="fixed">
+  </xacro:macro>
+</robot>
+	<!-- <joint name="gyro_joint" type="fixed">
 	    <axis xyz="0 1 0" />
 	    <origin xyz="0 0 0.04" rpy="0 0 0" />
@@ -170,5 +180,3 @@
 	    </inertial>
 	  </link>
-	<!--<sim_imu/> -->
-  </xacro:macro>
-</robot>
+	  <sim_imu/> -->

File: description/sensors_gazebo.urdf.xacro (robot description, xacro)
@@ -17,5 +17,5 @@
 <!-- Can't get this to work, will try the real camera -->
 	<xacro:macro name="sim_kinetic">
-		<gazebo reference="camera_link">
+		<!-- <gazebo reference="camera_link">
 		<material>Gazebo/Red</material>
 			<sensor type="depth" name="camera">
@@ -54,5 +54,33 @@
 				</plugin>
 			</sensor>
-		</gazebo>
+		</gazebo> -->
+		<gazebo reference="laser_frame">
+        <material>Gazebo/Black</material>
+        <sensor name="laser" type="ray">
+            <pose> 0 0 0 0 0 0 </pose>
+            <visualize>false</visualize>
+            <update_rate>10</update_rate>
+            <ray>
+                <scan>
+                    <horizontal>
+                        <samples>360</samples>
+                        <min_angle>-3.14</min_angle>
+                        <max_angle>3.14</max_angle>
+                    </horizontal>
+                </scan>
+                <range>
+                    <min>0.3</min>
+                    <max>12</max>
+                </range>
+            </ray>
+            <plugin name="laser_controller" filename="libgazebo_ros_ray_sensor.so">
+                <ros>
+                    <argument>~/out:=scan</argument>
+                </ros>
+                <output_type>sensor_msgs/LaserScan</output_type>
+                <frame_name>laser_frame</frame_name>
+            </plugin>
+        </sensor>
+    </gazebo>
 	</xacro:macro>
 </robot>
